Commit message: delete unnecessary parts

File: abb_irb120_gazebo/urdf/irb120_3_58_macro.xacro (robot description, xacro)
@@ -9,5 +9,5 @@
     <type>transmission_interface/SimpleTransmission</type>
     <joint name="${prefix}joint_1">
-      <hardwareInterface>PositionJointInterface</hardwareInterface>
+      <hardwareInterface>hardware_interface/PositionJointInterface</hardwareInterface>
     </joint>
     <actuator name="${prefix}motor1">
@@ -18,5 +18,5 @@
     <type>transmission_interface/SimpleTransmission</type>
     <joint name="${prefix}joint_2">
-      <hardwareInterface>PositionJointInterface</hardwareInterface>
+      <hardwareInterface>hardware_interface/PositionJointInterface</hardwareInterface>
     </joint>
     <actuator name="${prefix}motor2">
@@ -27,5 +27,5 @@
     <type>transmission_interface/SimpleTransmission</type>
     <joint name="${prefix}joint_3">
-      <hardwareInterface>PositionJointInterface</hardwareInterface>
+      <hardwareInterface>hardware_interface/PositionJointInterface</hardwareInterface>
     </joint>
     <actuator name="${prefix}motor3">
@@ -36,5 +36,5 @@
     <type>transmission_interface/SimpleTransmission</type>
     <joint name="${prefix}joint_4">
-      <hardwareInterface>PositionJointInterface</hardwareInterface>
+      <hardwareInterface>hardware_interface/PositionJointInterface</hardwareInterface>
     </joint>
     <actuator name="${prefix}motor4">
@@ -45,5 +45,5 @@
     <type>transmission_interface/SimpleTransmission</type>
     <joint name="${prefix}joint_5">
-      <hardwareInterface>PositionJointInterface</hardwareInterface>
+      <hardwareInterface>hardware_interface/PositionJointInterface</hardwareInterface>
     </joint>
     <actuator name="${prefix}motor5">
@@ -54,5 +54,5 @@
     <type>transmission_interface/SimpleTransmission</type>
     <joint name="${prefix}joint_6">
-      <hardwareInterface>PositionJointInterface</hardwareInterface>
+      <hardwareInterface>hardware_interface/PositionJointInterface</hardwareInterface>
     </joint>
     <actuator name="${prefix}motor6">

File: abb_irb120_support/urdf/irb120_3_58_macro.xacro (robot description, xacro)
@@ -197,5 +197,6 @@
       <parent link="${prefix}link_5"/>
       <child link="${prefix}link_6"/>
-      <limit effort="0" lower="-6.98132" upper="6.98132" velocity="7.33038"/>
+      <!--limit effort="0" lower="-6.98132" upper="6.98132" velocity="7.33038"/-->
+      <limit effort="0" lower="-3.14159" upper="3.14159" velocity="7.33038"/>
       <axis xyz="1 0 0"/>
       <dynamics damping="0.0" friction="0.0"/>
@@ -219,5 +220,5 @@
     <link name="${prefix}tool0" />
     <joint name="${prefix}link_6-tool0" type="fixed">
-      <origin xyz="0 0 0" rpy="0 ${radians(90)} 0" />
+      <origin xyz="0 0 0" rpy="0 0 0" />
       <parent link="${prefix}flange" />
       <child link="${prefix}tool0" />

File: abb_irb120_support/urdf/irb120t_3_58_macro.xacro (robot description, xacro)
@@ -219,5 +219,5 @@
     <link name="${prefix}tool0" />
     <joint name="${prefix}link_6-tool0" type="fixed">
-      <origin xyz="0 0 0" rpy="0 ${radians(90)} 0" />
+      <origin xyz="0 0 0" rpy="0 0 0" />
       <parent link="${prefix}flange" />
       <child link="${prefix}tool0" />
